File: Autonomous_robots/Eurobot_autonomous/Eurobot_autonomous.kicad_sch (KiCad schematic)
At the start: 17 parts, among them J1 Conn_01x02, J2 Conn_01x03, J3 Conn_01x03, J4 Conn_01x03, M1 Motor_Servo, M2 Motor_DC, M3 Motor_DC, SW1 SW_DIP_x01, U1 dc-dc_converter, U2 DRV8870DDA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

Commit message: PCB for autonomous robots updated
Connections:
- net GNDD: now also A1.29 (GND)
Changed lines of the file:
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@@
 (kicad_sch (version 20211123) (generator eeschema)
   (paper "A4" portrait)
+  (junction (at 99.06 127) (diameter 0) (color 0 0 0 0)
+  )
   (junction (at 55.88 26.67) (diameter 0) (color 0 0 0 0)
   )
@@
     (stroke (width 0) (type default) (color 0 0 0 0))
   )
+  (wire (pts (xy 99.06 128.27) (xy 99.06 127))
+    (stroke (width 0) (type default) (color 0 0 0 0))
+  )
   (wire (pts (xy 57.15 101.6) (xy 57.15 115.57))
     (stroke (width 0) (type default) (color 0 0 0 0))
@@
   )
   (wire (pts (xy 33.02 58.42) (xy 33.02 59.69))
+    (stroke (width 0) (type default) (color 0 0 0 0))
+  )
+  (wire (pts (xy 99.06 127) (xy 101.6 127))
     (stroke (width 0) (type default) (color 0 0 0 0))
   )
@@
     (pin "1")
   )
-  (symbol (lib_id "power:GNDD") (at 99.06 127 0) (unit 1)
-    (in_bom yes) (on_board yes) (fields_autoplaced)
-    (property "Reference" "#PWR013" (id 0) (at 99.06 133.35 0)
-      (effects (font (size 1.27 1.27)) hide)
-    )
-    (property "Value" "GNDD" (id 1) (at 99.06 132.08 0))
-    (property "Footprint" "" (id 2) (at 99.06 127 0)
-      (effects (font (size 1.27 1.27)) hide)
-    )
-    (property "Datasheet" "" (id 3) (at 99.06 127 0)
-      (effects (font (size 1.27 1.27)) hide)
-    )
+  (symbol (lib_id "power:GNDD") (at 99.06 128.27 0) (unit 1)
+    (in_bom yes) (on_board yes) (fields_autoplaced)
+    (property "Reference" "#PWR013" (id 0) (at 99.06 134.62 0)
+      (effects (font (size 1.27 1.27)) hide)
+    )
+    (property "Value" "GNDD" (id 1) (at 99.06 133.35 0))
+    (property "Footprint" "" (id 2) (at 99.06 128.27 0)
+      (effects (font (size 1.27 1.27)) hide)
+    )
+    (property "Datasheet" "" (id 3) (at 99.06 128.27 0)
+      (effects (font (size 1.27 1.27)) hide)
+    )

Commit message: wip
Connections:
- net at A1.14 (D11): now also U2.2 (IN2); no longer U2.3 (IN1)
- net at A1.15 (D12): now also U2.3 (IN1); no longer U2.2 (IN2)
Changed lines of the file:
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@@
   (junction (at 53.34 26.67) (diameter 0) (color 0 0 0 0)
   )
-  (wire (pts (xy 78.74 60.96) (xy 78.74 116.84))
+  (wire (pts (xy 76.2 114.3) (xy 77.47 114.3))
     (stroke (width 0) (type default) (color 0 0 0 0))
   )
@@
     (stroke (width 0) (type default) (color 0 0 0 0))
   )
-  (wire (pts (xy 76.2 114.3) (xy 86.36 114.3))
-    (stroke (width 0) (type default) (color 0 0 0 0))
-  )
   (wire (pts (xy 57.15 101.6) (xy 86.36 101.6))
     (stroke (width 0) (type default) (color 0 0 0 0))
@@
     (stroke (width 0) (type default) (color 0 0 0 0))
   )
+  (wire (pts (xy 86.36 114.3) (xy 78.74 114.3))
+    (stroke (width 0) (type default) (color 0 0 0 0))
+  )
   (wire (pts (xy 127 57.15) (xy 127 58.42))
     (stroke (width 0) (type default) (color 0 0 0 0))
@@
     (stroke (width 0) (type default) (color 0 0 0 0))
   )
-  (wire (pts (xy 78.74 116.84) (xy 86.36 116.84))
+  (wire (pts (xy 78.74 60.96) (xy 78.74 114.3))
     (stroke (width 0) (type default) (color 0 0 0 0))
   )
@@
     (stroke (width 0) (type default) (color 0 0 0 0))
   )
+  (wire (pts (xy 77.47 116.84) (xy 86.36 116.84))
+    (stroke (width 0) (type default) (color 0 0 0 0))
+  )
   (wire (pts (xy 142.24 104.14) (xy 142.24 102.87))
     (stroke (width 0) (type default) (color 0 0 0 0))
@@
     (stroke (width 0) (type default) (color 0 0 0 0))
   )
+  (wire (pts (xy 77.47 114.3) (xy 77.47 116.84))
+    (stroke (width 0) (type default) (color 0 0 0 0))
+  )
